File: Projects/ESC_rev01_1/CAN.kicad_sch (KiCad schematic)
At the start: 0 parts

Commit message: Update 07
Schematic is ready
INPUT PROTECTION schematic created
MOSFETs schematic created
CAN schematic created
FILTERs schematic created
MECHANICAL schematic created
STEP-DOWN schematic created
Footprints, 3D models are added and corrected (major issues)
Component placement started
Parts:
- added C52, C53: 60p, Capacitor_SMD:C_0603_1608Metric, symbol Device:C
- added C54: 2u2, Capacitor_SMD:C_0603_1608Metric, symbol Device:C
- added R44: 120R, Resistor_SMD:R_0603_1608Metric, symbol Device:R
- added R45, R46: 10R, Resistor_SMD:R_0603_1608Metric, symbol Device:R
- added R47: 10k, Resistor_SMD:R_0603_1608Metric, symbol Device:R
- added U6: Conn_01x04_2mnt, DF_ESC_rev01_1:CONN-SMD_S4B-XH-SM4-TB-LF-SN, symbol XH-2PWBPZ:Conn_01x04_2mnt
- added U7: ESDCAN24-2BLY, DF_ESC_rev01_1:SOT-23-3_L3.0-W1.7-P0.95-LS2.9-BR, symbol ESDCAN24-2BLY:ESDCAN24-2BLY
- added U8: 744227S, DF_ESC_rev01_1:FILTER-SMD_4P-L9.2-W6.0-P2.54-TL, symbol 744227S:744227S
- added U9: SN65HVD230, Package_SO:SOIC-8_3.9x4.9mm_P1.27mm, symbol Interface_CAN_LIN:SN65HVD230
Connections:
- new net: R47.1, U9.8 (Rs)
- new net: R45.2, U8.2
- new net: R46.2, U8.1
- new net +3V3: C54.1, U9.3 (VCC)
- new net +5V: U6.4
- new net CAN_N: U8.4, U9.6 (CANL)
- new net CAN_P: U8.3, U9.7 (CANH)
- new net CAN_RX: U9.4 (R)
- new net CAN_TX: U9.1 (D)
- new net C_CAN_N: C53.1, R44.2, R46.1, U6.2, U7.1
- new net C_CAN_P: C52.2, R44.1, R45.1, U6.3, U7.2
- new net GND: C52.1, C53.2, C54.2, R47.2, U6.1, U7.3, U9.2 (GND)
Other:
- note added: "BYPASS PLACE AS CLOSE AS POSSIBLE TO THE IC"
- note added: "MODE SELECTION RESISTOR SLEW RATE OF~15 V/us MORE INFO ON DATASHEET"
- note added: "[07] - CAN"

Commit message: Update 09
Components placement finished
Parts:
- J9: renamed from U6; symbol XH-2PWBPZ:Conn_01x04_2mnt -> DF_ESC_rev01_1:Conn_01x04_2mnt
- renumbered C52 to C50, C53 to C51, C54 to C52, R44 to R41, R45 to R42, R46 to R43, R47 to R44, U7 to U4, U8 to U5, U9 to U6
Changed lines of the file:
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@@
 		(dnp no)
 		(fields_autoplaced yes)
-		(property "Reference" "R44"
+		(property "Reference" "R41"
 			(at 109.22 100.3299 0)
 			(effects
@@
 			(project "ESC_rev01_1"
 				(path "/e63e39d7-6ac0-4ffd-8aa3-1841a4541b55/e32c040b-8a9b-40e1-ab88-651266d42ee1"
-					(reference "R44")
-					(unit 1)
-				)
-			)
-		)
-	)
-	(symbol
-		(lib_id "XH-2PWBPZ:Conn_01x04_2mnt")
+					(reference "R41")
+					(unit 1)
+				)
+			)
+		)
+	)
+	(symbol
+		(lib_id "DF_ESC_rev01_1:Conn_01x04_2mnt")
 		(at 66.04 104.14 180)
 		(unit 1)
@@
 		(dnp no)
 		(fields_autoplaced yes)
-		(property "Reference" "U6"
+		(property "Reference" "J9"
 			(at 60.96 100.3299 0)
 			(effects
@@
 			(project ""
 				(path "/e63e39d7-6ac0-4ffd-8aa3-1841a4541b55/e32c040b-8a9b-40e1-ab88-651266d42ee1"
-					(reference "U6")
+					(reference "J9")
 					(unit 1)
 				)
@@
 		(dnp no)
 		(fields_autoplaced yes)
-		(property "Reference" "#PWR076"
+		(property "Reference" "#PWR073"
 			(at 76.2 115.57 0)
 			(effects
@@
 			(project ""
 				(path "/e63e39d7-6ac0-4ffd-8aa3-1841a4541b55/e32c040b-8a9b-40e1-ab88-651266d42ee1"
-					(reference "#PWR076")
+					(reference "#PWR073")
 					(unit 1)
 				)
@@
 		(dnp no)
 		(fields_autoplaced yes)
-		(property "Reference" "#PWR081"
+		(property "Reference" "#PWR078"
 			(at 185.42 125.73 0)
 			(effects
@@
 			(project "ESC_rev01_1"
 				(path "/e63e39d7-6ac0-4ffd-8aa3-1841a4541b55/e32c040b-8a9b-40e1-ab88-651266d42ee1"
-					(reference "#PWR081")
+					(reference "#PWR078")
 					(unit 1)
 				)
@@
 		(dnp no)
 		(fields_autoplaced yes)
-		(property "Reference" "#PWR078"
+		(property "Reference" "#PWR075"
 			(at 106.68 129.54 0)
 			(effects
@@
 			(project "ESC_rev01_1"
 				(path "/e63e39d7-6ac0-4ffd-8aa3-1841a4541b55/e32c040b-8a9b-40e1-ab88-651266d42ee1"
-					(reference "#PWR078")
+					(reference "#PWR075")
 					(unit 1)
 				)
@@
 		(dnp no)
 		(fields_autoplaced yes)
-		(property "Reference" "#PWR080"
+		(property "Reference" "#PWR077"
 			(at 185.42 74.93 0)
 			(effects
@@
 			(project ""
 				(path "/e63e39d7-6ac0-4ffd-8aa3-1841a4541b55/e32c040b-8a9b-40e1-ab88-651266d42ee1"
-					(reference "#PWR080")
+					(reference "#PWR077")
 					(unit 1)
 				)
@@
 		(dnp no)
 		(fields_autoplaced yes)
-		(property "Reference" "R47"
+		(property "Reference" "R44"
 			(at 201.93 110.4899 0)
 			(effects
@@
 			(project "ESC_rev01_1"
 				(path "/e63e39d7-6ac0-4ffd-8aa3-1841a4541b55/e32c040b-8a9b-40e1-ab88-651266d42ee1"
-					(reference "R47")
+					(reference "R44")
 					(unit 1)
 				)
@@
 		(on_board yes)
 		(dnp no)
-		(property "Reference" "R45"
+		(property "Reference" "R42"
 			(at 125.476 86.614 90)
 			(effects
@@
 			(project "ESC_rev01_1"
 				(path "/e63e39d7-6ac0-4ffd-8aa3-1841a4541b55/e32c040b-8a9b-40e1-ab88-651266d42ee1"
-					(reference "R45")
+					(reference "R42")
 					(unit 1)
 				)
@@
 		(dnp no)
 		(fields_autoplaced yes)
-		(property "Reference" "#PWR082"
+		(property "Reference" "#PWR079"
 			(at 198.12 90.17 0)
 			(effects
@@
 			(project "ESC_rev01_1"
 				(path "/e63e39d7-6ac0-4ffd-8aa3-1841a4541b55/e32c040b-8a9b-40e1-ab88-651266d42ee1"
-					(reference "#PWR082")
+					(reference "#PWR079")
 					(unit 1)
 				)
@@
 		(dnp no)
 		(fields_autoplaced yes)
-		(property "Reference" "C53"
+		(property "Reference" "C51"
 			(at 110.49 116.8399 0)
 			(effects
@@
 			(project "ESC_rev01_1"
 				(path "/e63e39d7-6ac0-4ffd-8aa3-1841a4541b55/e32c040b-8a9b-40e1-ab88-651266d42ee1"
-					(reference "C53")
+					(reference "C51")
 					(unit 1)
 				)
@@
 		(dnp no)
 		(fields_autoplaced yes)
-		(property "Reference" "#PWR079"
+		(property "Reference" "#PWR076"
 			(at 111.76 80.01 0)
 			(effects
@@
 			(project "ESC_rev01_1"
 				(path "/e63e39d7-6ac0-4ffd-8aa3-1841a4541b55/e32c040b-8a9b-40e1-ab88-651266d42ee1"
-					(reference "#PWR079")
+					(reference "#PWR076")
 					(unit 1)
 				)
@@
 		(dnp no)
 		(fields_autoplaced yes)
-		(property "Reference" "#PWR075"
+		(property "Reference" "#PWR072"
 			(at 76.2 96.52 0)
 			(effects
@@
 			(project ""
 				(path "/e63e39d7-6ac0-4ffd-8aa3-1841a4541b55/e32c040b-8a9b-40e1-ab88-651266d42ee1"
-					(reference "#PWR075")
+					(reference "#PWR072")
 					(unit 1)
 				)
@@
 		(on_board yes)
 		(dnp no)
-		(property "Reference" "U8"
+		(property "Reference" "U5"
 			(at 143.256 93.218 0)
 			(effects
@@
 			(project ""
 				(path "/e63e39d7-6ac0-4ffd-8aa3-1841a4541b55/e32c040b-8a9b-40e1-ab88-651266d42ee1"
-					(reference "U8")
+					(reference "U5")
 					(unit 1)
 				)
@@
 		(dnp no)
 		(fields_autoplaced yes)
-		(property "Reference" "C52"
+		(property "Reference" "C50"
 			(at 110.49 83.8199 0)
 			(effects
@@
 			(project "ESC_rev01_1"
 				(path "/e63e39d7-6ac0-4ffd-8aa3-1841a4541b55/e32c040b-8a9b-40e1-ab88-651266d42ee1"
-					(reference "C52")
+					(reference "C50")
 					(unit 1)
 				)
@@
 		(on_board yes)
 		(dnp no)
-		(property "Reference" "U7"
+		(property "Reference" "U4"
 			(at 91.44 87.122 0)
 			(effects
@@
 			(project ""
 				(path "/e63e39d7-6ac0-4ffd-8aa3-1841a4541b55/e32c040b-8a9b-40e1-ab88-651266d42ee1"
-					(reference "U7")
+					(reference "U4")
 					(unit 1)
 				)
@@
 		(dnp no)
 		(fields_autoplaced yes)
-		(property "Reference" "#PWR083"
+		(property "Reference" "#PWR080"
 			(at 199.39 125.73 0)
 			(effects
@@
 			(project "ESC_rev01_1"
 				(path "/e63e39d7-6ac0-4ffd-8aa3-1841a4541b55/e32c040b-8a9b-40e1-ab88-651266d42ee1"
-					(reference "#PWR083")
+					(reference "#PWR080")
 					(unit 1)
 				)
@@
 		(dnp no)
 		(fields_autoplaced yes)
-		(property "Reference" "C54"
+		(property "Reference" "C52"
 			(at 201.93 77.4699 0)
 			(effects
@@
 			(project "ESC_rev01_1"
 				(path "/e63e39d7-6ac0-4ffd-8aa3-1841a4541b55/e32c040b-8a9b-40e1-ab88-651266d42ee1"
-					(reference "C54")
+					(reference "C52")
 					(unit 1)
 				)
@@
 		(on_board yes)
 		(dnp no)
-		(property "Reference" "U9"
+		(property "Reference" "U6"
 			(at 183.2767 90.17 0)
 			(effects
@@
 			(project ""
 				(path "/e63e39d7-6ac0-4ffd-8aa3-1841a4541b55/e32c040b-8a9b-40e1-ab88-651266d42ee1"
-					(reference "U9")
+					(reference "U6")
 					(unit 1)
 				)
@@
 		(dnp no)
 		(fields_autoplaced yes)
-		(property "Reference" "#PWR077"
+		(property "Reference" "#PWR074"
 			(at 97.79 109.22 0)
 			(effects
@@
 			(project "ESC_rev01_1"
 				(path "/e63e39d7-6ac0-4ffd-8aa3-1841a4541b55/e32c040b-8a9b-40e1-ab88-651266d42ee1"
-					(reference "#PWR077")
+					(reference "#PWR074")
 					(unit 1)
 				)
@@
 		(on_board yes)
 		(dnp no)
-		(property "Reference" "R46"
+		(property "Reference" "R43"
 			(at 125.476 106.934 90)
 			(effects
@@
 			(project "ESC_rev01_1"
 				(path "/e63e39d7-6ac0-4ffd-8aa3-1841a4541b55/e32c040b-8a9b-40e1-ab88-651266d42ee1"
-					(reference "R46")
-					(unit 1)
-				)
+					(reference "R43")
+					(unit 1)
+				)

Commit message: Update 11
Draft routing - diff signals and power
Connections:
- net R_CAN_P: now reaches R42.2, U5.2
- net R_CAN_N: now reaches R43.2, U5.1
Changed lines of the file:
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@@
+		)
+	)
+	(label "R_CAN_P"
+		(at 132.08 91.44 0)
+		(effects
+			(font
+				(size 1.27 1.27)
+			)
+			(justify left bottom)
+		)
+	)
+	(label "R_CAN_N"
+		(at 132.08 111.76 0)
+		(effects
+			(font
+				(size 1.27 1.27)
+			)
+			(justify left bottom)
 		)
 	)

Commit message: Update 01
Parts:
- C50, C51: value 60p -> C
- C52: value 2u2 -> C
- J9: footprint DF_ESC_rev01_1:CONN-SMD_S4B-XH-SM4-TB-LF-SN -> KeIr_lib:CONN-SMD_S4B-XH-SM4-TB-LF-SN; symbol DF_ESC_rev01_1:Conn_01x04_2mnt -> KeIr_sch_lib:Conn_01x04_2mnt
- R41: value 120R -> R
- R42, R43: value 10R -> R
- R44: value 10k -> R
- U4: footprint DF_ESC_rev01_1:SOT-23-3_L3.0-W1.7-P0.95-LS2.9-BR -> KeIr_lib:SOT-23-3_L3.0-W1.7-P0.95-LS2.9-BR
- U5: footprint DF_ESC_rev01_1:FILTER-SMD_4P-L9.2-W6.0-P2.54-TL -> KeIr_lib:FILTER-SMD_4P-L9.2-W6.0-P2.54-TL
Other:
- title: (none) -> DF_ESC_rev01_1
Changed lines of the file:
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@@
 	(generator_version "9.0")
 	(paper "A4")
+	(title_block
+		(title "DF_ESC_rev01_1")
+		(rev "01_1")
+		(comment 1 "Irina Kenko")
+		(comment 3 "irkenk8@gmail.com")
+		(comment 4 "Irina Kenko")
+		(comment 5 "irkenk8@gmail.com")
+	)
 	(text "MODE SELECTION RESISTOR\nSLEW RATE OF~15 V/us\n\nMORE INFO ON DATASHEET"
 		(exclude_from_sim no)
@@
 			)
 		)
-		(property "Value" "120R"
+		(property "Value" "R"
 			(at 109.22 102.8699 0)
 			(effects
@@
 	)
 	(symbol
-		(lib_id "DF_ESC_rev01_1:Conn_01x04_2mnt")
+		(lib_id "KeIr_sch_lib:Conn_01x04_2mnt")
 		(at 66.04 104.14 180)
 		(unit 1)
@@
 			)
 		)
-		(property "Footprint" "DF_ESC_rev01_1:CONN-SMD_S4B-XH-SM4-TB-LF-SN"
+		(property "Footprint" "KeIr_lib:CONN-SMD_S4B-XH-SM4-TB-LF-SN"
 			(at 66.04 89.154 0)
 			(effects
@@
 		(dnp no)
 		(fields_autoplaced yes)
-		(property "Reference" "#PWR073"
+		(property "Reference" "#PWR72"
 			(at 76.2 115.57 0)
 			(effects
@@
 			(project ""
 				(path "/e63e39d7-6ac0-4ffd-8aa3-1841a4541b55/e32c040b-8a9b-40e1-ab88-651266d42ee1"
-					(reference "#PWR073")
+					(reference "#PWR72")
 					(unit 1)
 				)
@@
 		(dnp no)
 		(fields_autoplaced yes)
-		(property "Reference" "#PWR078"
+		(property "Reference" "#PWR77"
 			(at 185.42 125.73 0)
 			(effects
@@
 			(project "ESC_rev01_1"
 				(path "/e63e39d7-6ac0-4ffd-8aa3-1841a4541b55/e32c040b-8a9b-40e1-ab88-651266d42ee1"
-					(reference "#PWR078")
+					(reference "#PWR77")
 					(unit 1)
 				)
@@
 		(dnp no)
 		(fields_autoplaced yes)
-		(property "Reference" "#PWR075"
+		(property "Reference" "#PWR74"
 			(at 106.68 129.54 0)
 			(effects
@@
 			(project "ESC_rev01_1"
 				(path "/e63e39d7-6ac0-4ffd-8aa3-1841a4541b55/e32c040b-8a9b-40e1-ab88-651266d42ee1"
-					(reference "#PWR075")
+					(reference "#PWR74")
 					(unit 1)
 				)
@@
 		(dnp no)
 		(fields_autoplaced yes)
-		(property "Reference" "#PWR077"
+		(property "Reference" "#PWR76"
 			(at 185.42 74.93 0)
 			(effects
@@
 			(project ""
 				(path "/e63e39d7-6ac0-4ffd-8aa3-1841a4541b55/e32c040b-8a9b-40e1-ab88-651266d42ee1"
-					(reference "#PWR077")
+					(reference "#PWR76")
 					(unit 1)
 				)
@@
 			)
 		)
-		(property "Value" "10k"
+		(property "Value" "R"
 			(at 201.93 113.0299 0)
 			(effects
@@
 			)
 		)
-		(property "Value" "10R"
+		(property "Value" "R"
 			(at 125.476 89.154 90)
 			(effects
@@
 		(dnp no)
 		(fields_autoplaced yes)
-		(property "Reference" "#PWR079"
+		(property "Reference" "#PWR78"
 			(at 198.12 90.17 0)
 			(effects
@@
 			(project "ESC_rev01_1"
 				(path "/e63e39d7-6ac0-4ffd-8aa3-1841a4541b55/e32c040b-8a9b-40e1-ab88-651266d42ee1"
-					(reference "#PWR079")
+					(reference "#PWR78")
 					(unit 1)
 				)
@@
 			)
 		)
-		(property "Value" "60p"
+		(property "Value" "C"
 			(at 110.49 119.3799 0)
 			(effects
@@
 		(dnp no)
 		(fields_autoplaced yes)
-		(property "Reference" "#PWR076"
+		(property "Reference" "#PWR75"
 			(at 111.76 80.01 0)
 			(effects
@@
 			(project "ESC_rev01_1"
 				(path "/e63e39d7-6ac0-4ffd-8aa3-1841a4541b55/e32c040b-8a9b-40e1-ab88-651266d42ee1"
-					(reference "#PWR076")
+					(reference "#PWR75")
 					(unit 1)
 				)
@@
 		(dnp no)
 		(fields_autoplaced yes)
-		(property "Reference" "#PWR072"
+		(property "Reference" "#PWR71"
 			(at 76.2 96.52 0)
 			(effects
@@
 			(project ""
 				(path "/e63e39d7-6ac0-4ffd-8aa3-1841a4541b55/e32c040b-8a9b-40e1-ab88-651266d42ee1"
-					(reference "#PWR072")
+					(reference "#PWR71")
 					(unit 1)
 				)
@@
 			)
 		)
-		(property "Footprint" "DF_ESC_rev01_1:FILTER-SMD_4P-L9.2-W6.0-P2.54-TL"
+		(property "Footprint" "KeIr_lib:FILTER-SMD_4P-L9.2-W6.0-P2.54-TL"
 			(at 143.51 111.76 0)
 			(effects
@@
 			)
 		)
-		(property "Value" "60p"
+		(property "Value" "C"
 			(at 110.49 86.3599 0)
 			(effects
@@
 			)
 		)
-		(property "Footprint" "DF_ESC_rev01_1:SOT-23-3_L3.0-W1.7-P0.95-LS2.9-BR"
+		(property "Footprint" "KeIr_lib:SOT-23-3_L3.0-W1.7-P0.95-LS2.9-BR"
 			(at 91.44 111.76 0)
 			(effects
@@
 		(dnp no)
 		(fields_autoplaced yes)
-		(property "Reference" "#PWR080"
+		(property "Reference" "#PWR79"
 			(at 199.39 125.73 0)
 			(effects
@@
 			(project "ESC_rev01_1"
 				(path "/e63e39d7-6ac0-4ffd-8aa3-1841a4541b55/e32c040b-8a9b-40e1-ab88-651266d42ee1"
-					(reference "#PWR080")
+					(reference "#PWR79")
 					(unit 1)
 				)
@@
 			)
 		)
-		(property "Value" "2u2"
+		(property "Value" "C"
 			(at 201.93 80.0099 0)
 			(effects
@@
 		(dnp no)
 		(fields_autoplaced yes)
-		(property "Reference" "#PWR074"
+		(property "Reference" "#PWR73"
 			(at 97.79 109.22 0)
 			(effects
@@
 			(project "ESC_rev01_1"
 				(path "/e63e39d7-6ac0-4ffd-8aa3-1841a4541b55/e32c040b-8a9b-40e1-ab88-651266d42ee1"
-					(reference "#PWR074")
+					(reference "#PWR73")
 					(unit 1)
 				)
@@
 			)
 		)
-		(property "Value" "10R"
+		(property "Value" "R"
 			(at 125.476 109.474 90)
 			(effects
