File: Projects/ESC_rev01_1/FILTERS.kicad_sch (KiCad schematic)
At the start: 0 parts

Commit message: Update 07
Schematic is ready
INPUT PROTECTION schematic created
MOSFETs schematic created
CAN schematic created
FILTERs schematic created
MECHANICAL schematic created
STEP-DOWN schematic created
Footprints, 3D models are added and corrected (major issues)
Component placement started
Parts:
- added C55, C56, C57, C58: 4n7, Capacitor_SMD:C_0603_1608Metric, symbol Device:C
- added C59, C60, C61, C62: 100n, Capacitor_SMD:C_0603_1608Metric, symbol Device:C
- added R48, R49, R50: 2k2, Resistor_SMD:R_0603_1608Metric, symbol Device:R
- added R51, R52, R53, R54: 10k, Resistor_SMD:R_0603_1608Metric, symbol Device:R
- added R55: 0R, Resistor_SMD:R_0603_1608Metric, symbol Device:R
- added U10: Conn_01x04_2mnt, DF_ESC_rev01_1:CONN-SMD_6P-P2.50_DEALON_XH-6PWB, symbol XH-2PWBPZ:Conn_01x06_2mnt
Connections:
- new net +3V3: C59.1, C60.1, C61.1, C62.1, R48.1, R49.1, R50.1, R51.1
- new net +5V: U10.6
- new net GND: C55.2, C56.2, C57.2, C58.2, C59.2, C60.2, C61.2, C62.2, U10.1
- new net HALL_1_IN: C55.1, R48.2, R52.1, U10.4
- new net HALL_1_OUT: R52.2
- new net HALL_2_IN: C56.1, R49.2, R53.1, U10.3
- new net HALL_2_OUT: R53.2
- new net HALL_3_IN: C57.1, R50.2, R54.1, U10.2
- new net HALL_3_OUT: R54.2
- new net TEMP_IN: C58.1, R51.2, R55.1, U10.5
- new net TEMP_MOTOR: R55.2
Other:
- note added: "HALL ENCODER INPUT"
- note added: "HALL ENCODER OUTPUT"
- note added: "HALL_1 FILTER"
- note added: "HALL_2 FILTER"
- note added: "HALL_3 FILTER"
- note added: "TEMP_MOTOR FILTER"
- note added: "TO MCU =>"
- note added: "[08] - FILTERS"

Commit message: Update 09
Components placement finished
Parts:
- renumbered C55 to C53, C56 to C54, C57 to C55, C58 to C56, C59 to C57, C60 to C58, C61 to C59, C62 to C60, U10 to J10, R48 to R45, R49 to R46, R50 to R47, R51 to R48, R52 to R49, R53 to R50, R54 to R51, R55 to R52

Commit message: Update 01
Parts:
- removed J10: Conn_01x04_2mnt, DF_ESC_rev01_1:CONN-SMD_6P-P2.50_DEALON_XH-6PWB, symbol XH-2PWBPZ:Conn_01x06_2mnt
- added J10: Conn_01x06_2mnt, KeIr_lib:CONN_DEALON_XH-6PWB, symbol DF_ESC_rev01_1:Conn_01x06_2mnt
- C53, C54, C55, C56: value 4n7 -> C
- C57, C58, C59, C60: value 100n -> C
- R45, R46, R47: value 2k2 -> R
- R48, R49, R50, R51: value 10k -> R
- R52: value 0R -> R
Connections:
- net +5V: now also J10.1
- net GND: now also J10.6
- net HALL_1_IN: now also J10.3
- net HALL_2_IN: now also J10.4
- net HALL_3_IN: now also J10.5
- net TEMP_IN: now also J10.2
Other:
- title: (none) -> DF_ESC_rev01_1
