File: Projects/ESC_rev01_1/INPUT PROTECTION.kicad_sch (KiCad schematic)
At the start: 13 parts, among them U1 XT30PW-M, U2 XH-2PWBPZ

Commit message: Update 09
Components placement finished
Parts:
- J1: renamed from U1; symbol XT30PW-M:XT30PW-M -> DF_ESC_rev01_1:XT30PW-M
- renumbered C63 to C3, U2 to J2, R67 to R1, TH2 to TH1
Changed lines of the file:
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@@
 	)
 	(symbol
-		(lib_id "XT30PW-M:XT30PW-M")
+		(lib_id "DF_ESC_rev01_1:XT30PW-M")
 		(at 46.99 71.12 270)
 		(mirror x)
@@
 		(on_board yes)
 		(dnp no)
-		(property "Reference" "U1"
+		(property "Reference" "J1"
 			(at 47.752 65.786 90)
 			(effects
@@
 		)
 		(property "Datasheet" "https://cn.bing.com/search?q=datasheet: XT30PW-M"
-			(at 47.117 73.406 0)
-			(effects
-				(font
-					(size 1.27 1.27)
-				)
-				(justify left)
+			(at 38.862 71.12 0)
+			(effects
+				(font
+					(size 1.27 1.27)
+				)
 				(hide yes)
 			)
@@
 		)
 		(property "LCSC" "C431092"
-			(at 46.99 71.12 0)
+			(at 40.64 71.374 0)
 			(effects
 				(font
@@
 			(project ""
 				(path "/e63e39d7-6ac0-4ffd-8aa3-1841a4541b55/62292eba-a192-4583-8aea-d56ef9bebcec"
-					(reference "U1")
+					(reference "J1")
 					(unit 1)
 				)
@@
 		(on_board yes)
 		(dnp no)
-		(property "Reference" "U2"
+		(property "Reference" "J2"
 			(at 109.982 127 0)
 			(effects
@@
 			(project ""
 				(path "/e63e39d7-6ac0-4ffd-8aa3-1841a4541b55/62292eba-a192-4583-8aea-d56ef9bebcec"
-					(reference "U2")
+					(reference "J2")
 					(unit 1)
 				)
@@
 		(dnp no)
 		(fields_autoplaced yes)
-		(property "Reference" "#PWR0109"
+		(property "Reference" "#PWR05"
 			(at 129.54 144.78 0)
 			(effects
@@
 			(project "ESC_rev01_1"
 				(path "/e63e39d7-6ac0-4ffd-8aa3-1841a4541b55/62292eba-a192-4583-8aea-d56ef9bebcec"
-					(reference "#PWR0109")
+					(reference "#PWR05")
 					(unit 1)
 				)
@@
 		(on_board yes)
 		(dnp no)
-		(property "Reference" "#PWR0110"
+		(property "Reference" "#PWR06"
 			(at 138.43 127 0)
 			(effects
@@
 			(project "ESC_rev01_1"
 				(path "/e63e39d7-6ac0-4ffd-8aa3-1841a4541b55/62292eba-a192-4583-8aea-d56ef9bebcec"
-					(reference "#PWR0110")
+					(reference "#PWR06")
 					(unit 1)
 				)
@@
 		(on_board yes)
 		(dnp no)
-		(property "Reference" "#PWR0108"
+		(property "Reference" "#PWR04"
 			(at 129.54 115.57 0)
 			(effects
@@
 			(project "ESC_rev01_1"
 				(path "/e63e39d7-6ac0-4ffd-8aa3-1841a4541b55/62292eba-a192-4583-8aea-d56ef9bebcec"
-					(reference "#PWR0108")
+					(reference "#PWR04")
 					(unit 1)
 				)
@@
 		(dnp no)
 		(fields_autoplaced yes)
-		(property "Reference" "C63"
+		(property "Reference" "C3"
 			(at 142.24 115.5699 0)
 			(effects
@@
 			(project "ESC_rev01_1"
 				(path "/e63e39d7-6ac0-4ffd-8aa3-1841a4541b55/62292eba-a192-4583-8aea-d56ef9bebcec"
-					(reference "C63")
+					(reference "C3")
 					(unit 1)
 				)
@@
 		(on_board yes)
 		(dnp no)
-		(property "Reference" "TH2"
+		(property "Reference" "TH1"
 			(at 122.682 130.81 0)
 			(effects
@@
 			(project "ESC_rev01_1"
 				(path "/e63e39d7-6ac0-4ffd-8aa3-1841a4541b55/62292eba-a192-4583-8aea-d56ef9bebcec"
-					(reference "TH2")
+					(reference "TH1")
 					(unit 1)
 				)
@@
 		(on_board yes)
 		(dnp no)
-		(property "Reference" "R67"
+		(property "Reference" "R1"
 			(at 126.492 117.094 0)
 			(effects
@@
 			(project "ESC_rev01_1"
 				(path "/e63e39d7-6ac0-4ffd-8aa3-1841a4541b55/62292eba-a192-4583-8aea-d56ef9bebcec"
-					(reference "R67")
-					(unit 1)
-				)
+					(reference "R1")
+					(unit 1)
+				)

Commit message: Update 01
Parts:
- C1, C2: footprint DF_ESC_rev01_1:CAP-TH_BD16.0-P7.50-D1.2-FD -> KeIr_lib:CAPPRD750W80D1600H2500; symbol LKMI2501K821MF:LKMI2501K821MF -> KeIr_sch_lib:LKMI2501K821MF
- C3, C4: value 100n -> C
- D1: footprint DF_ESC_rev01_1:SMA_L4.4-W2.8-LS5.1-BI -> KeIr_lib:SMA_L4.4-W2.8-LS5.1-BI
- D2: value LED_G -> LED
- J1: value XT30PW-M -> Conn_01x02_2mnt; footprint DF_ESC_rev01_1:CONN-TH_XT30PW-M -> KeIr_lib:CONN-TH_XT30PW-M; symbol DF_ESC_rev01_1:XT30PW-M -> KeIr_sch_lib:Conn_01x02_2mnt
- J2: footprint DF_ESC_rev01_1:CONN-SMD_XH-2PWBPZ -> KeIr_lib:CONN-SMD_XH-2PWBPZ
- R1, R3: value 2k2 -> R
- R2, R4: value 39k -> R
- TH1: value 10k -> Thermistor_NTC
Connections:
- net +3V3: now also TH1.1; no longer R1.2
- net ADC_TEMP: now also R1.2, TH1.2; no longer R1.1, TH1.1
- net GND: now also R1.1; no longer TH1.2
Other:
- title: (none) -> DF_ESC_rev01_1
- moved on the sheet: R1, TH1
Changed lines of the file:
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@@
 	(generator_version "9.0")
 	(paper "A4")
+	(title_block
+		(title "DF_ESC_rev01_1")
+		(rev "01_1")
+		(comment 1 "Irina Kenko")
+		(comment 3 "irkenk8@gmail.com")
+		(comment 4 "Irina Kenko")
+		(comment 5 "irkenk8@gmail.com")
+	)
 	(text "ESD \nSURGE PROTECTION"
 		(exclude_from_sim no)
@@
 			)
 		)
-		(property "Value" "LED_G"
+		(property "Value" "LED"
 			(at 209.55 89.2174 90)
 			(effects
@@
 		(dnp no)
 		(fields_autoplaced yes)
-		(property "Reference" "#PWR08"
+		(property "Reference" "#PWR8"
 			(at 205.74 64.77 0)
 			(effects
@@
 			(project "ESC_rev01_1"
 				(path "/e63e39d7-6ac0-4ffd-8aa3-1841a4541b55/62292eba-a192-4583-8aea-d56ef9bebcec"
-					(reference "#PWR08")
+					(reference "#PWR8")
 					(unit 1)
 				)
@@
 	)
 	(symbol
-		(lib_id "DF_ESC_rev01_1:XT30PW-M")
+		(lib_id "KeIr_sch_lib:Conn_01x02_2mnt")
 		(at 46.99 71.12 270)
 		(mirror x)
@@
 			)
 		)
-		(property "Value" "XT30PW-M"
+		(property "Value" "Conn_01x02_2mnt"
 			(at 54.61 76.962 90)
 			(effects
@@
 			)
 		)
-		(property "Footprint" "DF_ESC_rev01_1:CONN-TH_XT30PW-M"
+		(property "Footprint" "KeIr_lib:CONN-TH_XT30PW-M"
 			(at 36.83 71.12 0)
 			(effects
@@
 			)
 		)
-		(property "Datasheet" "https://cn.bing.com/search?q=datasheet: XT30PW-M"
+		(property "Datasheet" "https://jlcpcb.com/partdetail/Changzhou_AmassElec-XT30PW_M30_GY/C431092"
 			(at 38.862 71.12 0)
 			(effects
@@
 		(dnp no)
 		(property "Reference" "J2"
-			(at 109.982 127 0)
-			(effects
-				(font
-					(size 1.27 1.27)
-				)
-				(justify left)
+			(at 108.966 128.016 0)
+			(effects
+				(font
+					(size 1.27 1.27)
+				)
 			)
 		)
 		(property "Value" "XH-2PWBPZ"
-			(at 109.982 129.54 0)
-			(effects
-				(font
-					(size 1.27 1.27)
-				)
-				(justify left)
-			)
-		)
-		(property "Footprint" "DF_ESC_rev01_1:CONN-SMD_XH-2PWBPZ"
+			(at 104.14 130.81 0)
+			(effects
+				(font
+					(size 1.27 1.27)
+				)
+			)
+		)
+		(property "Footprint" "KeIr_lib:CONN-SMD_XH-2PWBPZ"
 			(at 114.3 138.43 0)
 			(effects
@@
 			)
 		)
-		(property "Footprint" "DF_ESC_rev01_1:SMA_L4.4-W2.8-LS5.1-BI"
+		(property "Footprint" "KeIr_lib:SMA_L4.4-W2.8-LS5.1-BI"
 			(at 87.63 74.93 0)
 			(effects
@@
 		(dnp no)
 		(fields_autoplaced yes)
-		(property "Reference" "#PWR03"
+		(property "Reference" "#PWR3"
 			(at 120.65 96.52 0)
 			(effects
@@
 			(project "ESC_rev01_1"
 				(path "/e63e39d7-6ac0-4ffd-8aa3-1841a4541b55/62292eba-a192-4583-8aea-d56ef9bebcec"
-					(reference "#PWR03")
+					(reference "#PWR3")
 					(unit 1)
 				)
@@
 			)
 		)
-		(property "Value" "100n"
+		(property "Value" "C"
 			(at 168.91 88.8999 0)
 			(effects
@@
 		(dnp no)
 		(fields_autoplaced yes)
-		(property "Reference" "#PWR05"
+		(property "Reference" "#PWR5"
 			(at 129.54 144.78 0)
 			(effects
@@
 			(project "ESC_rev01_1"
 				(path "/e63e39d7-6ac0-4ffd-8aa3-1841a4541b55/62292eba-a192-4583-8aea-d56ef9bebcec"
-					(reference "#PWR05")
+					(reference "#PWR5")
 					(unit 1)
 				)
@@
 		(dnp no)
 		(fields_autoplaced yes)
-		(property "Reference" "#PWR01"
+		(property "Reference" "#PWR1"
 			(at 52.07 64.77 0)
 			(effects
@@
 			(project ""
 				(path "/e63e39d7-6ac0-4ffd-8aa3-1841a4541b55/62292eba-a192-4583-8aea-d56ef9bebcec"
-					(reference "#PWR01")
+					(reference "#PWR1")
 					(unit 1)
 				)
@@
 		(on_board yes)
 		(dnp no)
-		(property "Reference" "#PWR06"
+		(property "Reference" "#PWR6"
 			(at 138.43 127 0)
 			(effects
@@
 			(project "ESC_rev01_1"
 				(path "/e63e39d7-6ac0-4ffd-8aa3-1841a4541b55/62292eba-a192-4583-8aea-d56ef9bebcec"
-					(reference "#PWR06")
+					(reference "#PWR6")
 					(unit 1)
 				)
@@
 		(on_board yes)
 		(dnp no)
-		(property "Reference" "#PWR04"
+		(property "Reference" "#PWR4"
 			(at 129.54 115.57 0)
 			(effects
@@
 			(project "ESC_rev01_1"
 				(path "/e63e39d7-6ac0-4ffd-8aa3-1841a4541b55/62292eba-a192-4583-8aea-d56ef9bebcec"
-					(reference "#PWR04")
+					(reference "#PWR4")
 					(unit 1)
 				)
@@
 			)
 		)
-		(property "Value" "100n"
+		(property "Value" "C"
 			(at 142.24 118.1099 0)
 			(effects
@@
 			)
 		)
-		(property "Value" "2k2"
+		(property "Value" "R"
 			(at 152.146 89.154 0)
 			(effects
@@
 	)
 	(symbol
-		(lib_id "LKMI2501K821MF:LKMI2501K821MF")
+		(lib_id "KeIr_sch_lib:LKMI2501K821MF")
 		(at 116.84 82.55 0)
 		(unit 1)
@@
 		(dnp no)
 		(property "Reference" "C1"
-			(at 109.728 82.55 0)
-			(effects
-				(font
-					(size 1.27 1.27)
-				)
-				(justify left)
+			(at 113.284 81.534 0)
+			(effects
+				(font
+					(size 1.27 1.27)
+				)
 			)
 		)
 		(property "Value" "LKMI2501K821MF"
-			(at 98.552 85.09 0)
-			(effects
-				(font
-					(size 1.27 1.27)
-				)
-				(justify left)
-			)
-		)
-		(property "Footprint" "DF_ESC_rev01_1:CAP-TH_BD16.0-P7.50-D1.2-FD"
+			(at 106.172 83.566 0)
+			(effects
+				(font
+					(size 1.27 1.27)
+				)
+			)
+		)
+		(property "Footprint" "KeIr_lib:CAPPRD750W80D1600H2500"
 			(at 116.84 92.71 0)
 			(effects
@@
 			)
 		)
-		(property "Datasheet" "https://item.szlcsc.com/48887.html"
+		(property "Datasheet" "https://jlcpcb.com/partdetail/Ymin-LKMI2501K821MF/C443097"
 			(at 116.84 94.742 0)
 			(effects
@@
 	(symbol
 		(lib_id "Device:Thermistor_NTC")
-		(at 129.54 132.08 0)
+		(at 129.54 118.11 0)
 		(unit 1)
 		(exclude_from_sim no)
@@
 		(dnp no)
 		(property "Reference" "TH1"
-			(at 122.682 130.81 0)
+			(at 122.682 116.84 0)
 			(effects
 				(font
@@
 			)
 		)
-		(property "Value" "10k"
-			(at 122.682 133.35 0)
+		(property "Value" "Thermistor_NTC"
+			(at 122.682 119.38 0)
 			(effects
 				(font
@@
 		)
 		(property "Footprint" "Resistor_SMD:R_0603_1608Metric"
-			(at 129.54 130.81 0)
+			(at 129.54 116.84 0)
 			(effects
 				(font
@@
 		)
 		(property "Datasheet" "~"
-			(at 129.54 130.81 0)
+			(at 129.54 116.84 0)
 			(effects
 				(font
@@
 		)
 		(property "Description" "Temperature dependent resistor, negative temperature coefficient"
-			(at 129.54 132.08 0)
+			(at 129.54 118.11 0)
 			(effects
 				(font
@@
 		(dnp no)
 		(fields_autoplaced yes)
-		(property "Reference" "#PWR09"
+		(property "Reference" "#PWR9"
 			(at 205.74 97.79 0)
 			(effects
@@
 			(project "ESC_rev01_1"
 				(path "/e63e39d7-6ac0-4ffd-8aa3-1841a4541b55/62292eba-a192-4583-8aea-d56ef9bebcec"
-					(reference "#PWR09")
+					(reference "#PWR9")
 					(unit 1)
 				)
@@
 		(dnp no)
 		(fields_autoplaced yes)
-		(property "Reference" "#PWR02"
+		(property "Reference" "#PWR2"
 			(at 57.15 88.9 0)
 			(effects
@@
 			(project ""
 				(path "/e63e39d7-6ac0-4ffd-8aa3-1841a4541b55/62292eba-a192-4583-8aea-d56ef9bebcec"
-					(reference "#PWR02")
+					(reference "#PWR2")
 					(unit 1)
 				)
@@
 		(on_board yes)
 		(dnp no)
-		(property "Reference" "#PWR07"
+		(property "Reference" "#PWR7"
 			(at 157.48 99.06 0)
 			(effects
@@
 			(project "ESC_rev01_1"
 				(path "/e63e39d7-6ac0-4ffd-8aa3-1841a4541b55/62292eba-a192-4583-8aea-d56ef9bebcec"
-					(reference "#PWR07")
+					(reference "#PWR7")
 					(unit 1)
 				)
@@
 	(symbol
 		(lib_id "Device:R")
-		(at 129.54 118.11 180)
+		(at 129.54 132.08 180)
 		(unit 1)
 		(exclude_from_sim no)
@@
 		(dnp no)
 		(property "Reference" "R1"
-			(at 126.492 117.094 0)
-			(effects
-				(font
-					(size 1.27 1.27)
-				)
-			)
-		)
-		(property "Value" "2k2"
-			(at 126.238 119.38 0)
+			(at 126.492 131.064 0)
+			(effects
+				(font
+					(size 1.27 1.27)
+				)
+			)
+		)
+		(property "Value" "R"
+			(at 126.238 133.35 0)
 			(effects
 				(font
@@
 		)
 		(property "Footprint" "Resistor_SMD:R_0603_1608Metric"
-			(at 131.318 118.11 90)
+			(at 131.318 132.08 90)
 			(effects
 				(font
@@
 		)
 		(property "Datasheet" "~"
-			(at 129.54 118.11 0)
+			(at 129.54 132.08 0)
 			(effects
 				(font
@@
 		)
 		(property "Description" "Resistor"
-			(at 129.54 118.11 0)
+			(at 129.54 132.08 0)
 			(effects
 				(font
@@
 	)
 	(symbol
-		(lib_id "LKMI2501K821MF:LKMI2501K821MF")
+		(lib_id "KeIr_sch_lib:LKMI2501K821MF")
 		(at 124.46 82.55 0)
 		(unit 1)
@@
 		(dnp no)
 		(property "Reference" "C2"
-			(at 127.508 82.55 0)
-			(effects
-				(font
-					(size 1.27 1.27)
-				)
-				(justify left)
+			(at 128.524 81.534 0)
+			(effects
+				(font
+					(size 1.27 1.27)
+				)
 			)
 		)
 		(property "Value" "LKMI2501K821MF"
-			(at 125.73 85.344 0)
-			(effects
-				(font
-					(size 1.27 1.27)
-				)
-				(justify left)
-			)
-		)
-		(property "Footprint" "DF_ESC_rev01_1:CAP-TH_BD16.0-P7.50-D1.2-FD"
+			(at 135.636 83.312 0)
+			(effects
+				(font
+					(size 1.27 1.27)
+				)
+			)
+		)
+		(property "Footprint" "KeIr_lib:CAPPRD750W80D1600H2500"
 			(at 124.46 92.71 0)
 			(effects
@@
 			)
 		)
-		(property "Datasheet" "https://item.szlcsc.com/48887.html"
+		(property "Datasheet" "https://jlcpcb.com/partdetail/Ymin-LKMI2501K821MF/C443097"
 			(at 124.46 94.742 0)
 			(effects
@@
 			)
 		)
-		(property "Value" "39k"
+		(property "Value" "R"
 			(at 160.02 78.7399 0)
 			(effects
@@
 			)
 		)
-		(property "Value" "39k"
+		(property "Value" "R"
 			(at 208.28 78.7399 0)
 			(effects
