File: Projects/ESC_rev01_1/MCU.kicad_sch (KiCad schematic)
At the start: 36 parts, among them J3 XH-2PWBPZ, J4 Conn_01x06, J5 Conn_01x03, SW1 PTS526SK15SMTR2LFS, U2 STM32F405RGTx, Y1 8M 10ppm X50328MSB2GI

Commit message: Update 01
Parts:
- removed J4: Conn_01x06, DF_ESC_rev01_1:CONN-SMD_6P-P2.50_DEALON_XH-6PWB, symbol XH-2PWBPZ:Conn_01x06_2mnt
- added J4: Conn_01x06_2mnt, KeIr_lib:CONN_DEALON_XH-6PWB, symbol DF_ESC_rev01_1:Conn_01x06_2mnt
- C10, C11, C12, C13, C16, C17, C19, C21, C23: value 100n -> C
- C14, C15: value 10p -> C
- C18, C20: value 2u2 -> C
- C22: value 1u -> C
- C9: value 10u -> C
- D11: value LED_R -> LED
- D6: footprint DF_ESC_rev01_1:D_SOD-882_BI -> KeIr_lib:D_SOD-882_BI
- D8: value LED_G -> LED
- J3: value XH-2PWBPZ -> Conn_01x08_2mnt; footprint DF_ESC_rev01_1:CONN-SMD_8P-P2.50_HX25003-8AWB -> KeIr_lib:CONN-SMD_8P-P2.50_HX25003-8AWB; symbol DF_ESC_rev01_1:Conn_01x08_2mnt -> KeIr_sch_lib:Conn_01x08_2mnt
- J5: value Conn_01x03 -> Conn_01x03_2mnt; footprint DF_ESC_rev01_1:CONN-SMD_XH-3AWB -> KeIr_lib:CONN-SMD_XH-3AWB
- R10: value 1k -> R
- R11, R13: value 2k2 -> R
- R12: value 100R -> R
- R7: renamed from R8; value 0R -> R
- R8: renamed from R9; value 0R -> R
- R9: renamed from R7; value 1k -> R
- SW1: value PTS526SK15SMTR2LFS -> SW_DIP_x01_4pin; footprint DF_ESC_rev01_1:SW-SMD_4P-L5.2-W5.2-P3.70-LS6.4 -> KeIr_lib:SW-SMD_4P-L5.2-W5.2-P3.70-LS6.4
- Y1: value 8M 10ppm X50328MSB2GI -> Crystal; footprint DF_ESC_rev01_1:CRYSTAL-SMD_L5.0-W3.2 -> KeIr_lib:CRYSTAL-SMD_L5.0-W3.2
Connections:
- net +3V3_DBG: now also J4.1
- net GND: now also J4.3, J4.5
- net NRST: now also J4.6
- net SWCLK: now also J4.4
- net SWDIO: now also J4.2
Other:
- note added: "NRST internally pulled-up (The reset network protects the device against parasitic resets.)"
- note added: "external clock source"
- note added: "ferrite bead is crutial for optimal filtering effectiveness (only in analog section - could resonate LC)"
- note added: "or to 3V3?"
- note removed: "NRST internally pulled-up"
- title: (none) -> DF_ESC_rev01_1
- moved on the sheet: D8, R9
