File: Projects/ESC_rev01_1/MECHANICAL.kicad_sch (KiCad schematic)
At the start: 0 parts

Commit message: Update 07
Schematic is ready
INPUT PROTECTION schematic created
MOSFETs schematic created
CAN schematic created
FILTERs schematic created
MECHANICAL schematic created
STEP-DOWN schematic created
Footprints, 3D models are added and corrected (major issues)
Component placement started
Parts:
- added H1, H2, H3, H4: MountingHole_Pad, MountingHole:MountingHole_3.2mm_M3_DIN965_Pad, symbol Mechanical:MountingHole_Pad
- added R63, R64, R65, R66: 0R, Resistor_SMD:R_0603_1608Metric, symbol Device:R
Connections:
- new net: H2.1, R64.1
- new net: H4.1, R66.1
- new net: H1.1, R63.1
- new net: H3.1, R65.1
- new net GND: R63.2, R64.2, R65.2, R66.2
Other:
- note added: "FIT A ZERO OHM LINK, CAP OR RESISTOR"
- note added: "LABELS"
- note added: "LOGOS"
- note added: "MOUNTING HOLES"
- note added: "PCB"
- note added: "[10] - MECHANICAL"

Commit message: Update 09
Components placement finished
Parts:
- renumbered R63 to R60, R64 to R61, R65 to R62, R66 to R63
Other:
- note added: "- THERMISTOR MOVED TO LOWER LEG OF THE ADC PIN - BOOT PIN PULLED-DOWN TO GND - CHANGED BULCK CAPACITANCE - CHANGE PHASE SENSE RRESISTORS - CHANGED NETS SENSE PHASES TO DIFFERENTIAL PAIRS - INVERTED TX AND RX CONNECTOR PI"
- note added: "MODIFICATION FROM VESC 4.11:"
- moved on the sheet: H1, H2, H3, H4, R60, R61, R62, R63

Commit message: Update 01
Parts:
- R60, R61, R62, R63: value 0R -> R
Other:
- title: (none) -> DF_ESC_rev01_1
Changed lines of the file:
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@@
 	(generator_version "9.0")
 	(paper "A4")
+	(title_block
+		(title "DF_ESC_rev01_1")
+		(rev "01_1")
+		(comment 1 "Irina Kenko")
+		(comment 3 "irkenk8@gmail.com")
+		(comment 4 "Irina Kenko")
+		(comment 5 "irkenk8@gmail.com")
+	)
 	(rectangle
 		(start 227.33 54.61)
@@
 			)
 		)
-		(property "Value" "0R"
+		(property "Value" "R"
 			(at 130.81 113.0299 0)
 			(effects
@@
 			)
 		)
-		(property "Value" "0R"
+		(property "Value" "R"
 			(at 130.81 82.5499 0)
 			(effects
@@
 			)
 		)
-		(property "Value" "0R"
+		(property "Value" "R"
 			(at 176.53 113.0299 0)
 			(effects
@@
 		(dnp no)
 		(fields_autoplaced yes)
-		(property "Reference" "#PWR0100"
+		(property "Reference" "#PWR99"
 			(at 128.27 93.98 0)
 			(effects
@@
 			(project "ESC_rev01_1"
 				(path "/e63e39d7-6ac0-4ffd-8aa3-1841a4541b55/f0db8fa9-4626-4d2b-9dd9-5c3f1156b21e"
-					(reference "#PWR0100")
+					(reference "#PWR99")
 					(unit 1)
 				)
@@
 			)
 		)
-		(property "Value" "0R"
+		(property "Value" "R"
 			(at 176.53 82.5499 0)
 			(effects
@@
 		(dnp no)
 		(fields_autoplaced yes)
-		(property "Reference" "#PWR0102"
+		(property "Reference" "#PWR101"
 			(at 173.99 93.98 0)
 			(effects
@@
 			(project "ESC_rev01_1"
 				(path "/e63e39d7-6ac0-4ffd-8aa3-1841a4541b55/f0db8fa9-4626-4d2b-9dd9-5c3f1156b21e"
-					(reference "#PWR0102")
+					(reference "#PWR101")
 					(unit 1)
 				)
@@
 		(dnp no)
 		(fields_autoplaced yes)
-		(property "Reference" "#PWR0103"
+		(property "Reference" "#PWR102"
 			(at 173.99 124.46 0)
 			(effects
@@
 			(project "ESC_rev01_1"
 				(path "/e63e39d7-6ac0-4ffd-8aa3-1841a4541b55/f0db8fa9-4626-4d2b-9dd9-5c3f1156b21e"
-					(reference "#PWR0103")
+					(reference "#PWR102")
 					(unit 1)
 				)
@@
 		(dnp no)
 		(fields_autoplaced yes)
-		(property "Reference" "#PWR0101"
+		(property "Reference" "#PWR100"
 			(at 128.27 124.46 0)
 			(effects
@@
 			(project "ESC_rev01_1"
 				(path "/e63e39d7-6ac0-4ffd-8aa3-1841a4541b55/f0db8fa9-4626-4d2b-9dd9-5c3f1156b21e"
-					(reference "#PWR0101")
+					(reference "#PWR100")
 					(unit 1)
 				)
