File: Projects/ESC_rev01_1/MOSFETs.kicad_sch (KiCad schematic)
At the start: 0 parts

Commit message: Update 07
Schematic is ready
INPUT PROTECTION schematic created
MOSFETs schematic created
CAN schematic created
FILTERs schematic created
MECHANICAL schematic created
STEP-DOWN schematic created
Footprints, 3D models are added and corrected (major issues)
Component placement started
Parts:
- added C50: 2u2, Capacitor_SMD:C_0603_1608Metric, symbol Device:C
- added C51: 2n2, Capacitor_SMD:C_0603_1608Metric, symbol Device:C
- added J4, J5, J6: Conn_01x01, DF_ESC_rev01_1:WE_7461084, symbol Connector_Generic:Conn_01x01
- added NT1, NT2, NT3, NT4, NT5, NT6, NT7, NT8: NetTie_2, NetTie:NetTie-2_SMD_Pad2.0mm, symbol Device:NetTie_2
- added Q1, Q2, Q3, Q4, Q5, Q6: HSBA15810C, Package_SO:PowerPAK_SO-8_Single, symbol DF_ESC_rev01_1:HSBA15810C
- added R29, R30, R35, R36, R41, R42: 4R7, Resistor_SMD:R_0603_1608Metric, symbol Device:R
- added R31, R32, R37, R38: 100R, Resistor_SMD:R_0603_1608Metric, symbol Device:R
- added R33, R39, R43: 39k, Resistor_SMD:R_0603_1608Metric, symbol Device:R
- added R34, R40: 0R001, Resistor_SMD:R_0603_1608Metric, symbol Device:R
Connections:
- new net +VDC: Q1.5 (D), Q3.5 (D), Q5.5 (D)
- new net GND: NT3.1, NT6.1, NT8.1, R33.2, R39.2, R43.2
- new net H1_LOW: NT2.2, Q2.1 (S), Q2.2 (S), Q2.3 (S)
- new net H1_VS: NT1.1
- new net H2_LOW: NT5.2, Q4.1 (S), Q4.2 (S), Q4.3 (S)
- new net H2_VS: NT4.1
- new net H3_LOW: NT8.2, Q6.1 (S), Q6.2 (S), Q6.3 (S)
- new net H3_VS: NT7.1
- new net M_H1: R29.1
- new net M_H1_RG: Q1.4 (G), R29.2
- new net M_H2: R35.1
- new net M_H2_RG: Q3.4 (G), R35.2
- new net M_H3: R41.1
- new net M_H3_RG: Q5.4 (G), R41.2
- new net M_L1: R30.1
- new net M_L1_RG: Q2.4 (G), R30.2, R33.1
- new net M_L2: R36.1
- new net M_L2_RG: Q4.4 (G), R36.2, R39.1
- new net M_L3: R42.1
- new net M_L3_RG: Q6.4 (G), R42.2, R43.1
- new net PHASE_1: J4.1 (Pin_1), NT1.2, Q1.1 (S), Q1.2 (S), Q1.3 (S), Q2.5 (D)
- new net PHASE_2: J5.1 (Pin_1), NT4.2, Q3.1 (S), Q3.2 (S), Q3.3 (S), Q4.5 (D)
- new net PHASE_3: J6.1 (Pin_1), NT7.2, Q5.1 (S), Q5.2 (S), Q5.3 (S), Q6.5 (D)
- new net S1_N: C50.1, R31.1
- new net S1_P: C50.2, R32.1
- new net S2_N: C51.1, R37.1
- new net S2_P: C51.2, R38.1
- new net SH1_N: NT2.1, R31.2, R34.1
- new net SH1_P: NT3.2, R32.2, R34.2
- new net SH2_N: NT5.1, R37.2, R40.1
- new net SH2_P: NT6.2, R38.2, R40.2
Other:
- note added: "Hx_VS"
- note added: "MCU SENSING FEEDBACK"
- note added: "OUTPUT PHASE 1"
- note added: "OUTPUT PHASE 2"
- note added: "OUTPUT PHASE 3"
- note added: "PHASE 1"
- note added: "PHASE 2"
- note added: "PHASE 3"
- note added: "PLACE AS CLOSE AS POSSIBLE TO THE BULK CAPACITANCE"
- note added: "Q_CONTROL"
- note added: "Q_SOURCES"
- note added: "ROUTE AS KELVING CONNECTIONS"
- note added: "SENSE 1"
- note added: "SENSE 2"
- note added: "[06] - MOSFETs"

Commit message: Update 09
Components placement finished
Parts:
- NT1, NT4, NT7: footprint NetTie:NetTie-2_SMD_Pad2.0mm -> NetTie:NetTie-2_SMD_Pad0.5mm
- NT2, NT3, NT5, NT6, NT8: footprint NetTie:NetTie-2_SMD_Pad2.0mm -> DF_ESC_rev01_1:NetTie-2_SMD_Pad_4.0x2.0mm
- Q1, Q2, Q3, Q4, Q5, Q6: footprint Package_SO:PowerPAK_SO-8_Single -> DF_ESC_rev01_1:PQFN-8_L6.0-W5.0-P1.27-LS6.0-BL
- R31: renamed from R34; footprint Resistor_SMD:R_0603_1608Metric -> DF_ESC_rev01_1:RES_VISHAY_WSLP27261L000; symbol Device:R -> DF_ESC_rev01_1:R_Shunt
- R37: renamed from R40; footprint Resistor_SMD:R_0603_1608Metric -> DF_ESC_rev01_1:RES_VISHAY_WSLP27261L000; symbol Device:R -> DF_ESC_rev01_1:R_Shunt
- renumbered C50 to C48, C51 to C49, J4 to J6, J5 to J7, J6 to J8, R29 to R26, R30 to R27, R31 to R28, R32 to R29, R33 to R30, R35 to R32, R36 to R33, R37 to R34, R38 to R35, R39 to R36, R41 to R38, R42 to R39, R43 to R40
Connections:
- net SH1_N: now also R31.2; no longer R31.1
- net SH1_P: now also R31.1; no longer R31.2
- net SH2_N: now also R37.2; no longer R37.1
- net SH2_P: now also R37.1; no longer R37.2

Commit message: Update 01
Parts:
- C48: value 2u2 -> C
- C49: value 2n2 -> C
- J6, J7, J8: footprint DF_ESC_rev01_1:WE_7461084 -> KeIr_lib:WE_7461084
- NT3: renamed from NT2; footprint DF_ESC_rev01_1:NetTie-2_SMD_Pad_4.0x2.0mm -> KeIr_lib:NetTie-2_SMD_Pad_4.0x2.0mm
- NT4: renamed from NT3; footprint DF_ESC_rev01_1:NetTie-2_SMD_Pad_4.0x2.0mm -> KeIr_lib:NetTie-2_SMD_Pad_4.0x2.0mm
- NT6: renamed from NT5; footprint DF_ESC_rev01_1:NetTie-2_SMD_Pad_4.0x2.0mm -> KeIr_lib:NetTie-2_SMD_Pad_4.0x2.0mm
- NT7: renamed from NT6; footprint DF_ESC_rev01_1:NetTie-2_SMD_Pad_4.0x2.0mm -> KeIr_lib:NetTie-2_SMD_Pad_4.0x2.0mm
- NT9: renamed from NT8; footprint DF_ESC_rev01_1:NetTie-2_SMD_Pad_4.0x2.0mm -> KeIr_lib:NetTie-2_SMD_Pad_4.0x2.0mm
- Q1, Q2, Q3, Q4, Q5, Q6: footprint DF_ESC_rev01_1:PQFN-8_L6.0-W5.0-P1.27-LS6.0-BL -> KeIr_lib:PQFN-8_L6.0-W5.0-P1.27-LS6.0-BL
- R26, R27, R32, R33, R38, R39: value 4R7 -> R
- R28, R29, R34, R35: value 100R -> R
- R30, R36, R40: value 39k -> R
- R31, R37: footprint DF_ESC_rev01_1:RES_VISHAY_WSLP27261L000 -> KeIr_lib:RES_VISHAY_WSLP27261L000
- renumbered NT1 to NT2, NT4 to NT5, NT7 to NT8
Other:
- note added: "AVOID INTERFERENCE PRODUCED BY NEARBY MOSFETS"
- note added: "GATE RESISTOR"
- note added: "PULL-DOWN RESISTOR"
- note added: "ROUTE AS DIFF PAIR TO BETTER CONTROL NOISE"
- title: (none) -> DF_ESC_rev01_1
