File: Projects/ESC_rev01_1/STEP-DOWN.kicad_sch (KiCad schematic)
At the start: 10 parts, among them U3 AMS1117-3.3

Commit message: Update 09
Components placement finished
Parts:
- renumbered U3 to U1
Other:
- note added: "[03] - STEP DOWN"
- moved on the sheet: C5, C6, C7, C8, D3, D4, D5, R5, R6, U1

Commit message: Update 01
Parts:
- C5, C6: value 1u -> C
- C7, C8: value 1u -> C; MPN (none) -> CL10A105KP8NNNC
- D3, D5: value LED_G -> LED
- R5, R6: value 1k -> R
Other:
- title: (none) -> DF_ESC_rev01_1
Changed lines of the file:
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@@
 	(generator_version "9.0")
 	(paper "A4")
+	(title_block
+		(title "DF_ESC_rev01_1")
+		(rev "01_1")
+		(comment 1 "Irina Kenko")
+		(comment 3 "irkenk8@gmail.com")
+		(comment 4 "Irina Kenko")
+		(comment 5 "irkenk8@gmail.com")
+	)
 	(text "FROM MOSFET DRIVER\nOR EXTERNAL"
 		(exclude_from_sim no)
@@
 		(dnp no)
 		(fields_autoplaced yes)
-		(property "Reference" "#PWR010"
+		(property "Reference" "#PWR10"
 			(at 97.79 85.09 0)
 			(effects
@@
 			(project "ESC_rev01_1"
 				(path "/e63e39d7-6ac0-4ffd-8aa3-1841a4541b55/c73e4030-1bb6-4559-8c3c-f52e48758511"
-					(reference "#PWR010")
+					(reference "#PWR10")
 					(unit 1)
 				)
@@
 			)
 		)
-		(property "Value" "1u"
+		(property "Value" "C"
 			(at 162.56 96.5199 0)
 			(effects
@@
 			)
 		)
+		(property "MPN" "CL10A105KP8NNNC "
+			(at 158.75 95.25 0)
+			(effects
+				(font
+					(size 1.27 1.27)
+				)
+				(hide yes)
+			)
+		)
 		(pin "2"
 		)
@@
 		(dnp no)
 		(fields_autoplaced yes)
-		(property "Reference" "#PWR014"
+		(property "Reference" "#PWR14"
 			(at 163.83 109.22 0)
 			(effects
@@
 			(project "ESC_rev01_1"
 				(path "/e63e39d7-6ac0-4ffd-8aa3-1841a4541b55/c73e4030-1bb6-4559-8c3c-f52e48758511"
-					(reference "#PWR014")
+					(reference "#PWR14")
 					(unit 1)
 				)
@@
 		(on_board yes)
 		(dnp no)
-		(property "Reference" "#FLG02"
+		(property "Reference" "#FLG2"
 			(at 198.12 88.265 0)
 			(effects
@@
 			(project "ESC_rev01_1"
 				(path "/e63e39d7-6ac0-4ffd-8aa3-1841a4541b55/c73e4030-1bb6-4559-8c3c-f52e48758511"
-					(reference "#FLG02")
+					(reference "#FLG2")
 					(unit 1)
 				)
@@
 		(dnp no)
 		(fields_autoplaced yes)
-		(property "Reference" "#PWR015"
+		(property "Reference" "#PWR15"
 			(at 204.47 85.09 0)
 			(effects
@@
 			(project "ESC_rev01_1"
 				(path "/e63e39d7-6ac0-4ffd-8aa3-1841a4541b55/c73e4030-1bb6-4559-8c3c-f52e48758511"
-					(reference "#PWR015")
+					(reference "#PWR15")
 					(unit 1)
 				)
@@
 			)
 		)
-		(property "Value" "LED_G"
+		(property "Value" "LED"
 			(at 101.6 106.9974 90)
 			(effects
@@
 		(dnp no)
 		(fields_autoplaced yes)
-		(property "Reference" "#PWR011"
+		(property "Reference" "#PWR11"
 			(at 97.79 116.84 0)
 			(effects
@@
 			(project "ESC_rev01_1"
 				(path "/e63e39d7-6ac0-4ffd-8aa3-1841a4541b55/c73e4030-1bb6-4559-8c3c-f52e48758511"
-					(reference "#PWR011")
+					(reference "#PWR11")
 					(unit 1)
 				)
@@
 		(dnp no)
 		(fields_autoplaced yes)
-		(property "Reference" "#PWR013"
+		(property "Reference" "#PWR13"
 			(at 146.05 109.22 0)
 			(effects
@@
 			(project "ESC_rev01_1"
 				(path "/e63e39d7-6ac0-4ffd-8aa3-1841a4541b55/c73e4030-1bb6-4559-8c3c-f52e48758511"
-					(reference "#PWR013")
+					(reference "#PWR13")
 					(unit 1)
 				)
@@
 		(on_board yes)
 		(dnp no)
-		(property "Reference" "#FLG01"
+		(property "Reference" "#FLG1"
 			(at 105.41 88.265 0)
 			(effects
@@
 			(project "ESC_rev01_1"
 				(path "/e63e39d7-6ac0-4ffd-8aa3-1841a4541b55/c73e4030-1bb6-4559-8c3c-f52e48758511"
-					(reference "#FLG01")
+					(reference "#FLG1")
 					(unit 1)
 				)
@@
 			)
 		)
-		(property "Value" "1u"
+		(property "Value" "C"
 			(at 173.99 96.5199 0)
 			(effects
@@
 		)
 		(property "Description" "Unpolarized capacitor"
+			(at 170.18 95.25 0)
+			(effects
+				(font
+					(size 1.27 1.27)
+				)
+				(hide yes)
+			)
+		)
+		(property "MPN" "CL10A105KP8NNNC "
 			(at 170.18 95.25 0)
 			(effects
@@
 			)
 		)
-		(property "Value" "1u"
+		(property "Value" "C"
 			(at 120.65 96.5199 0)
 			(effects
@@
 			)
 		)
-		(property "Value" "1k"
+		(property "Value" "R"
 			(at 100.33 96.5199 0)
 			(effects
@@
 			)
 		)
-		(property "Value" "LED_G"
+		(property "Value" "LED"
 			(at 208.28 106.9974 90)
 			(effects
@@
 		(dnp no)
 		(fields_autoplaced yes)
-		(property "Reference" "#PWR016"
+		(property "Reference" "#PWR16"
 			(at 204.47 116.84 0)
 			(effects
@@
 			(project "ESC_rev01_1"
 				(path "/e63e39d7-6ac0-4ffd-8aa3-1841a4541b55/c73e4030-1bb6-4559-8c3c-f52e48758511"
-					(reference "#PWR016")
+					(reference "#PWR16")
 					(unit 1)
 				)
@@
 		(dnp no)
 		(fields_autoplaced yes)
-		(property "Reference" "#PWR012"
+		(property "Reference" "#PWR12"
 			(at 121.92 109.22 0)
 			(effects
@@
 			(project "ESC_rev01_1"
 				(path "/e63e39d7-6ac0-4ffd-8aa3-1841a4541b55/c73e4030-1bb6-4559-8c3c-f52e48758511"
-					(reference "#PWR012")
+					(reference "#PWR12")
 					(unit 1)
 				)
@@
 			)
 		)
-		(property "Value" "1u"
+		(property "Value" "C"
 			(at 132.08 96.5199 0)
 			(effects
@@
 			)
 		)
-		(property "Value" "1k"
+		(property "Value" "R"
 			(at 207.01 96.5199 0)
 			(effects
